Commit message: otonom surus eski halinde waypointlerle çalıştırılmaya calısıldı, fsm eklendi

File: install/robotanik_sim/share/robotanik_sim/urdf/robotanik.urdf (robot description, URDF)
Before this commit: robot robotanik, 10 links, 9 joints
Links:
- link base_link: geometry collision box size=0.40 0.30 0.325; visual box size=0.40 0.30 0.325
Joints:
- joint left_wheel_joint: origin xyz=-0.15 0.146 -0.1525 rpy=-1.5708 0 0 -> xyz=-0.135 0.121 -0.1525 rpy=-1.5708 0 0
- joint right_wheel_joint: origin xyz=-0.15 -0.146 -0.1525 rpy=1.5708 0 0 -> xyz=-0.135 -0.121 -0.1525 rpy=1.5708 0 0
- joint sonar_back_joint: origin xyz=-0.26 0 0.05 rpy=0 0 3.14159 -> xyz=-0.21 0 0.05 rpy=0 0 3.14159
- joint sonar_front_center_joint: origin xyz=0.26 0 0.05 rpy=0 0 0 -> xyz=0.21 0 0.05 rpy=0 0 0
- joint sonar_front_left_joint: origin xyz=0.26 0.15 0.05 rpy=0 0 0.52 -> xyz=0.21 0.125 0.05 rpy=0 0 0.698
- joint sonar_front_right_joint: origin xyz=0.26 -0.15 0.05 rpy=0 0 -0.52 -> xyz=0.21 -0.125 0.05 rpy=0 0 -0.698
